File: Brunei_Brain.brd (EAGLE design)
At the start: 100 x 70 mm, 78 parts, among them IC1 4098D, T1 BC846, T2 BC846, U1 USD-SOCKETNEW, U3 HEX_CONVERTER, Y2 CSTCE16M0V53-R0 16MHZ

Commit message: Started v2 update process.
Parts:
- removed U$9: MICRO-FIT_3.0_4POS_VERT_THRU, Schuyler:MICRO-FIT_3.0_4POS_VERT_THROUGH
- added U$15: MICRO-FIT_3.0_5POS_VERT_THRU, Schuyler:MICRO-FIT_3.0_5POS_VERT_THROUGH
- C13, C14, C15, C16, C17: value 0.1 uF -> 0.1uF
- JP2: value (none) -> M023.5MM
- U$2: value CC3-4805SF-ECC3-4805SF-E -> CC3-4805SF-E"
- U3: device SparkFun:SO016 -> SparkFun-DigitalIC:SO016
Connections:
- net 3.3V renamed 3V3
- new net SPEC_TRIGGER: U$15.P$5
- net +5V: now also U$15.P$1; no longer JP1.6, U$9.P$1
- net ARDUINO_V: now also JP1.6
- net GND: now also U$15.P$2; no longer U$9.P$2
- net RX_FROM_SPEC: now also U$15.P$4; no longer U$9.P$4
- net TX_TO_SPEC: now also U$15.P$3; no longer U$9.P$3
Routing:
- net MOSI_IO11: track 88.6 -> 89.1 mm
- net SCK_IO13: track 90.8 -> 91.3 mm
- net +5V: track 201.5 -> 201.0 mm
- net N$163: track 35.0 -> 35.6 mm
- net N$8: track 33.1 -> 33.6 mm

Commit message: some continuing updates
Parts:
- removed JP1: (no value), pinhead:1X07
- added C21: 0.1uF, resistor:C0603
- added R22: 10k, SparkFun-Passives:0603-RES
- added U$20: BATTERY_12MM, Schuyler:KEYSTONE_12MM_BATT_SM
- added U2: DS3234, Schuyler:SOIC-20_MAXIM
- C10, C12: value 4.7 uF -> 4.7uF
- R3, R4, R5, R6: value (none) -> DNP
- R8: value (none) -> 20k
- U$1: value CC6-4812SF-ECC6-4812SF-E -> CC6-4812SF-E'
- moved U$15 88.6 mm to (60.5, 67.8)
Connections:
- removed net +5V: C12.1, C13.1, C16.1, C2.1, C8.1, IC1.16, IC1.3, IC1.5, R10.2, R5.2, R9.2, TP6.TP, U$10.P$1, U$15.P$1, U$2.P$7, U$4.4, U$6.P$1, U$7.2, U$8.P$1, U$8.P$3
- new net 5V0: C12.1, C13.1, C16.1, C2.1, C8.1, IC1.16, R5.2, R9.2, TP6.TP, U$10.P$1, U$15.P$1, U$2.P$7, U$4.4, U$6.P$1, U$7.2, U$8.P$1, U$8.P$3
- new net N$20: R3.1, R4.2, U$1.P$6
- net 12V: now also R3.2; no longer R3.1
- net ARDUINO_V: now also C21.1, IC1.16, IC1.3, IC1.5, R10.2, R22.2, U2.P$4; no longer JP1.6
- net GND: now also C21.2, U$20.P$3, U2.P$10, U2.P$11, U2.P$12, U2.P$13, U2.P$14, U2.P$15, U2.P$2, U2.P$7, U2.P$8, U2.P$9; no longer JP1.7
- net IO3: now also R22.1, U2.P$5; no longer JP1.5
- net IO9: now also U2.P$1; no longer JP1.1
- net MISO_IO12: now also U2.P$19; no longer JP1.3
- net MOSI_IO11: now also U2.P$17; no longer JP1.2
- net N$6: now also U$20.P$1, U$20.P$2, U2.P$16; no longer R3.2, R4.2, U$1.P$6
- net SCK_IO13: now also U2.P$18, U2.P$20; no longer JP1.4
Routing:
- net +5V: track 201.0 -> 0.00 mm, vias 2 -> 0
- net 5V0: track 0.00 -> 191.7 mm, vias 0 -> 2
- net SCK_IO13: track 91.3 -> 79.5 mm
- net 12V: track 44.4 -> 37.3 mm
- net ARDUINO_V: track 85.8 -> 92.6 mm
- net IO9: track 17.4 -> 11.6 mm
- net MISO_IO12: track 90.9 -> 85.2 mm
- net N$6: track 5.06 -> 0.00 mm
- net MOSI_IO11: track 89.1 -> 85.8 mm
- net 3.7BATT: track 25.7 -> 23.0 mm

Commit message: Version 2.0 Complete
Parts:
- removed IC1: 4098D, 40xx:SO16
- removed JP2: M023.5MM, SparkFun-Connectors:SCREWTERMINAL-3.5MM-2
- removed U$1: CC6-4812SF-E', Schuyler:CC6-XXXXXF-E
- removed U$10: MICRO-FIT_3.0_7POS_VERT_THRU, Schuyler:MICRO-FIT_3.0_7POS_VERT_THROUGH
- removed U$11: GM1WA55321ACOMMON_CATHODE, Schuyler:0606_4PIN
- removed U$12, U$13: MICRO-FIT_3.0_2POS_VERT_THRU, Schuyler:MICRO-FIT_3.0_2POS_VERT_THROUGH
- removed U$14: MICRO-FIT_3.0_6POS_VERT_THRU, Schuyler:MICRO-FIT_3.0_6POS_VERT_THROUGH
- removed U$15: MICRO-FIT_3.0_5POS_VERT_THRU, Schuyler:MICRO-FIT_3.0_5POS_VERT_THROUGH
- removed U$2: CC3-4805SF-E", Schuyler:CC3-XXXXXF-E
- removed U$20: BATTERY_12MM, Schuyler:KEYSTONE_12MM_BATT_SM
- removed U$3: RF201L2S, Schuyler:SOD-106
- removed U$4: MCP73831/2, Schuyler:SOT23-5
- removed U$5, U$6: LSM115J, Schuyler:DO-214BA
- removed U$7: LM3480IM4, SparkFun-PowerIC:SOT23-3
- removed U$8: MAX3311, Schuyler:UMAX10_MAXIM
- removed Y2: CSTCE16M0V53-R0 16MHZ, SmartPrj:RESONATOR
- removed ZU4: ATMEGA328P-PU, SmartPrj:DIL28-3
- added B1: BATTERY_12MM, Schuyler:KEYSTONE_12MM_BATT_SM
- added C23, C24: 0.1uF, resistor:C0603
- added C25: 1uF, rcl:C1206
- added D1: RF201L2S, Schuyler:SOD-106
- added D3: LSM115J, Schuyler:DO-214BA
- added D4: RGB_LED_COMMON_ANODE_1, Schuyler:PLCC-4
- added J1: M023.5MM, SparkFun-Connectors:SCREWTERMINAL-3.5MM-2
- added J2, J3: MICRO-FIT_3.0_2POS_VERT_THRU, Schuyler:MICRO-FIT_3.0_2POS_VERT_THROUGH
- added J4: MICRO-FIT_3.0_7POS_VERT_THRU, Schuyler:MICRO-FIT_3.0_7POS_VERT_THROUGH
- added J5: MICRO-FIT_3.0_6POS_VERT_THRU, Schuyler:MICRO-FIT_3.0_6POS_VERT_THROUGH
- added J6: MICRO-FIT_3.0_5POS_VERT_THRU, Schuyler:MICRO-FIT_3.0_5POS_VERT_THROUGH
- added SD: MICRO_SD_DM3AT, Schuyler:MICROSD_DM3AT
- added U10: MULTIVIBRATOR_DUAL, Schuyler:SO-16_SSG
- added U4: CC6-4812SF-E', Schuyler:CC6-XXXXXF-E
- added U5: CC3-4805SF-E", Schuyler:CC3-XXXXXF-E
- added U6: HEX_CONVERTERS, Schuyler:SO-16_SSG
- added U8: ST232, Schuyler:SO-16_SSG
- added U9: ATMEGA328P-PU, SmartPrj:DIL28-3
- added Y1: CSTCE16M0V53-R0 16MHZ, SmartPrj:RESONATOR
- C1: value 1uF -> 4.7uF; device rcl:C1206 -> resistor:C0603
- C11: value 100n -> 0.1uF; device SmartPrj:C0603-ROUND -> rcl:C0603
- C12: value 4.7uF -> 1uF; device resistor:C0603 -> rcl:C1206
- C13: value 0.1uF -> 1uF; device resistor:C0603 -> rcl:C1206
- C14, C15: device resistor:C0603 -> rcl:C0603
- C18: value 1uF -> 0.1uF
- C19, C20: value 100nF -> 0.1uF; device rcl:C0603 -> resistor:C0603
- C2: value 1uF -> 0.1uF; device rcl:C1206 -> resistor:C0603
- C3, C4: value 1uF -> 0.1uF; device rcl:C1206 -> rcl:C0603
- C6, C7: value 0.1uF -> 1uF; device rcl:C0603 -> rcl:C1206
- C8: device rcl:C0603 -> resistor:C0603
- C9: value 100n -> 0.1uF; device SmartPrj:C0603-ROUND -> resistor:C0603
- D2: value CD1206-S01575 -> LSM115J; device diode:MINIMELF -> Schuyler:DO-214BA
- R1: value (none) -> 4.99M
- R10: value 10k -> DNP
- R11: value 600 -> DNP
- R12: value 400 -> DNP
- R13: value 420 -> DNP
- R14: value 4.99M -> 33k
- R15: value 100k -> 33k
- R16: value 250k -> 33k
- R17: value 75k -> 10k
- R18: value (none) -> 1M; device SparkFun-Passives:0603-RES -> SmartPrj:R0603-ROUND
- R19: value (none) -> 600
- R2: value (none) -> 100k
- R20: value (none) -> 360
- R21: value 10k -> 360
- R4: value DNP -> 10k
- R5, R6: value DNP -> 1k
- R7: value 1M -> 20k; device SmartPrj:R0603-ROUND -> SparkFun-Passives:0603-RES
- R8: value 20k -> 250k
- R9: value 100k -> 75k
- S1: value (none) -> DIP03YL
- U1: value USD-SOCKETNEW -> DS3234; device SparkFun:MICRO-SD-SOCKET-PP -> Schuyler:SOIC-20_MAXIM
- U2: value DS3234 -> LM3480IM4; device Schuyler:SOIC-20_MAXIM -> SparkFun-PowerIC:SOT23-3
- U3: value HEX_CONVERTER -> MCP73831/2; device SparkFun-DigitalIC:SO016 -> Schuyler:SOT23-5
- moved RESET 98.3 mm to (14.6, 3.56), turned to 180 degrees
- moved C16 67.6 mm to (11.4, 7.62), turned to 0 degrees
- moved C17 66.6 mm to (16.5, 7.62), turned to 0 degrees
- moved D2 62.2 mm to (60.5, 51.1), turned to 180 degrees
- moved C19 59.4 mm to (21.6, 7.62), turned to 0 degrees
- moved C1 56.9 mm to (56.9, 60.5), turned to 180 degrees
- moved TP4 56.7 mm to (16.2, 43.9), turned to 180 degrees
- moved U1 56.5 mm to (27.9, 58.4), turned to 90 degrees
- moved R16 53.7 mm to (47.0, 5.08)
- moved C12 51.3 mm to (52.6, 8.64), turned to 270 degrees
- moved R2 50.2 mm to (68.8, 57.4), turned to 0 degrees
- moved R17 49.8 mm to (10.3, 23.2), turned to 0 degrees
- moved R14 48.8 mm to (37.8, 5.08), turned to 0 degrees
- moved R13 47.8 mm to (54.1, 41.7), turned to 270 degrees
- moved C21 47.5 mm to (25.9, 23.2)
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Connections:
- removed net N$11: C15.1, U$8.P$8
- removed net N$12: C17.2, U$8.P$2
- removed net SPEC_TRIGGER: U$15.P$5
- new net N$19: C16.1, U8.1
- new net N$21: C16.2, U8.3
- new net N$22: C17.1, U8.4
- new net N$23: C17.2, U8.5
- new net N$24: C19.1, U8.6
- new net N$26: C18.2, U8.2
- net 12V: now also C12.1, C14.1, J5.P$1, R10.2, U4.P$7; no longer C1.1, C7.1, R3.2, U$1.P$7, U$14.P$1
- net 3.7BATT: now also D2.P$1, J3.P$1, R8.2, U3.3; no longer R16.2, U$13.P$1, U$4.3, U$5.P$1
- net 3V3: now also C8.1, SD.P$4, U2.1, U6.1; no longer C14.1, U$7.1, U1.4, U3.1
- net 48V: now also C7.1, D1.P$2, R1.2, U4.P$1, U5.P$1; no longer C3.1, R14.2, U$1.P$1, U$2.P$1, U$3.P$2
- net 48_V_BATTERY: now also D1.P$1, J1.1, J2.P$1; no longer JP2.1, U$12.P$1, U$3.P$1
- net 5V0: now also C1.1, C15.1, C18.1, C20.1, D3.P$1, J4.P$1, J6.P$1, R12.2, U2.2, U3.4, U5.P$7, U8.16; no longer C12.1, C16.1, C8.1, IC1.16, R5.2, R9.2, U$10.P$1, U$15.P$1, U$2.P$7, U$4.4, U$6.P$1, U$7.2, U$8.P$1, U$8.P$3
- net AD0: now also U6.3, U9.23; no longer R1.1, ZU4.23
- net AD1: now also U1.P$1, U9.24; no longer R2.1, ZU4.24
- net AD2: now also R21.2, U9.25; no longer R12.2, ZU4.25
- net AD3: now also R20.2, U9.26; no longer R13.2, ZU4.26
- net AD4/SDA: now also C3.1, R1.1, R2.2, U9.27; no longer C19.1, R14.1, R15.2, ZU4.27
- net AD5/SCL: now also C11.1, R8.1, R9.2, U9.28; no longer C20.1, R16.1, R17.2, ZU4.28
- net ARDUINO_V: now also C24.1, C9.1, D2.P$2, D3.P$2, D4.P$2, R17.2, R4.2, U1.P$4, U10.16, U10.3, U10.5, U9.20, U9.7; no longer C11.2, D2.C, IC1.16, IC1.3, IC1.5, R10.2, R21.2, U$5.P$2, U$6.P$2, U2.P$4, ZU4.20, ZU4.7
- net AREF: now also C23.2, U9.21; no longer C9.2, ZU4.21
- net DEUTERIUM_ENABLE: now also J5.P$4, R14.2; no longer R18.2, U$14.P$4
- net GND: now also B1.P$3, C11.2, C23.1, C24.2, C9.2, J1.2, J2.P$2, J3.P$2, J4.P$2, J5.P$2, J6.P$2, R11.1, R13.1, R14.1, R16.1, R2.1, R7.1, R9.1, SD.P$10, SD.P$11, SD.P$13, SD.P$14, SD.P$6, U1.P$10, U1.P$11, U1.P$12, U1.P$13, U1.P$14, U1.P$15, U1.P$2, U1.P$7, U1.P$8, U1.P$9, U10.13, U10.8, U2.3, U3.2, U4.P$3, U4.P$5, U5.P$3, U5.P$5, U6.8, U8.15, U9.22, U9.8, Y1.2; no longer C11.1, C16.2, C9.1, IC1.13, IC1.8, JP2.2, R17.1, R18.1, R19.1, R20.1, R4.1, R6.1, R8.1, U$1.P$3, U$1.P$5, U$10.P$2, U$11.P$4, U$12.P$2, U$13.P$2, U$14.P$2, U$15.P$2, U$2.P$3, U$2.P$5, U$20.P$3, U$4.2, U$7.3, U$8.P$10, U1.6, U1.CD1, U1.CD2, U1.GND1, U1.GND3, U2.P$10, U2.P$11, U2.P$12, U2.P$13, U2.P$14, U2.P$15, U2.P$2, U2.P$7, U2.P$8, U2.P$9, U3.8, Y2.2, ZU4.22, ZU4.8
- net IO2: now also J4.P$6, U9.4; no longer R9.1, U$4.1, ZU4.4
- net IO3: now also R3.2, R4.1, U1.P$5, U9.5; no longer R22.1, U2.P$5, ZU4.5
- net IO4: now also J6.P$5, U9.6; no longer U$10.P$5, ZU4.6
- net IO5: now also J4.P$5, U9.11; no longer U$10.P$6, ZU4.11
- net IO6: now also U10.4, U9.12; no longer IC1.4, ZU4.12
- net IO7: now also R19.2, U9.13; no longer R11.2, ZU4.13
- net IO8: now also R5.1, U9.14; no longer U3.3, ZU4.14
- net IO9: now also R6.1, U9.15; no longer U2.P$1, ZU4.15
- net LAMP_5V: now also J5.P$3; no longer U$14.P$3
- net MISO_IO12: now also SD.P$7, U1.P$19, U9.18; no longer U1.7, U2.P$19, ZU4.18
- net MOSI_IO11: now also J4.P$3, U1.P$17, U6.5, U9.17; no longer U$10.P$3, U2.P$17, U3.5, ZU4.17
- net N$1: now also T2.3, U5.P$2; no longer T1.3, U$2.P$2
- net N$10: now also R3.1, U3.1; no longer C17.1, U$8.P$9
- net N$13: now also C25.2, U10.1; no longer C18.2, IC1.1
- net N$14: now also C25.1, R22.1, U10.2; no longer C18.1, IC1.2, R10.1
- net N$15: now also D4.P$1, R19.1; no longer R11.1, U$11.P$1
- net N$16: now also J4.P$7; no longer U$10.P$7
- net N$163: now also SD.P$2, U6.2; no longer U1.2, U3.2
- net N$17: now also D4.P$4, R20.1; no longer R12.1, U$11.P$2
- net N$18: now also D4.P$3, R21.1; no longer R13.1, U$11.P$3
- net N$2: now also T1.3, U4.P$2; no longer T2.3, U$1.P$2
- net N$20: now also R10.1, R11.2, U4.P$6; no longer R3.1, R4.2, U$1.P$6
- net N$3: now also R5.2, T1.1; no longer R2.2, T2.1
- net N$4: now also R6.2, T2.1; no longer R1.2, T1.1
- net N$5: now also R12.1, R13.2, U5.P$6; no longer R5.1, R6.2, U$2.P$6
- net N$6: now also B1.P$1, B1.P$2, U1.P$16; no longer U$20.P$1, U$20.P$2, U2.P$16
- net N$7: now also R7.2, U3.5; no longer R8.2, U$4.5
- net N$8: now also SD.P$3, U6.4; no longer U1.3, U3.4
- net N$9: now also SD.P$5, U6.6; no longer U1.5, U3.6
- net RESET: now also R17.1, U10.7, U9.1; no longer D2.A, IC1.7, R21.1, ZU4.1
- net RX_FROM_SPEC: now also J6.P$4, U8.13; no longer U$15.P$4, U$8.P$6
- net RX_IO0: now also U8.12, U9.2; no longer U$8.P$5, ZU4.2
- net SCK_IO13: now also J4.P$4, U1.P$18, U1.P$20, U6.7, U9.19; no longer U$10.P$4, U2.P$18, U2.P$20, U3.7, ZU4.19
- net SHUTTER_ENABLE: now also J5.P$6, R16.2; no longer R20.2, U$14.P$6
- net SS_IO10: now also U9.16; no longer ZU4.16
- net TUNGSTEN_ENABLE: now also J5.P$5, R15.2; no longer R19.2, U$14.P$5
- net TX_IO1: now also U8.11, U9.3; no longer U$8.P$4, ZU4.3
- net TX_TO_SPEC: now also J6.P$3, U8.14; no longer U$15.P$3, U$8.P$7
- net XTAL1: now also R18.1, U9.9, Y1.3; no longer R7.1, Y2.3, ZU4.9
- net XTAL2: now also R18.2, U9.10, Y1.1; no longer R7.2, Y2.1, ZU4.10
Routing:
- net RX_IO0: track 122.9 -> 12.1 mm, vias 3 -> 0
- net AD3: track 116.9 -> 21.0 mm, vias 3 -> 0
- net GND: track 15.2 -> 106.1 mm, vias 2 -> 41
- net 3.7BATT: track 23.0 -> 99.2 mm, vias 1 -> 12
- net AD2: track 95.0 -> 21.4 mm, vias 3 -> 0
- net AD1: track 93.0 -> 20.5 mm
- net IO3: track 17.3 -> 88.5 mm, vias 1 -> 6
- net ARDUINO_V: track 92.6 -> 161.3 mm, vias 3 -> 7
- net RESET: track 155.0 -> 91.8 mm, vias 4 -> 0
- net TX_IO1: track 69.2 -> 11.6 mm, vias 3 -> 0
- net AD0: track 66.6 -> 10.2 mm, vias 1 -> 0
- net AD5/SCL: track 62.7 -> 9.78 mm, vias 2 -> 0
- net IO9: track 11.6 -> 54.5 mm, vias 2 -> 3
- net N$6: track 0.00 -> 36.9 mm, vias 0 -> 2
- net MISO_IO12: track 85.2 -> 50.2 mm, vias 3 -> 0
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- added copper zone on layer 1, net 48V
Other:
- board size 100 x 70 mm -> 88.9 x 69.8 mm
- board text added: "12V"
- board text added: "3.3V"
- board text added: "48V"
- board text added: "5V"
- board text added: "Batt"
- board text added: "GND"
- board text added: "LEDIF-PEAT v2.0 12/20/13"
- board text added: "S. Senft-Grupp, MIT"
- board text added: "UV/VIS Lamp"
- board text removed: "08/22/2012"
- board text removed: "Absorbance Lamp"
- board text removed: "Battery"
- board text removed: "LEDIF-PEAT v1.0"
- board text removed: "S. Senft-Grupp"

Commit message: Updated part attributes for ordering
Parts:
- R1: value 4.99M -> 5.1M
- R19: value 600 -> 604
- R8: value 250k -> 249k
