File: Brunei_Brain.sch (EAGLE design)
At the start: 78 parts, among them IC1 4098D, T1 BC846, T2 BC846, U1 USD-SOCKETNEW, U3 HEX_CONVERTER, Y2 CSTCE16M0V53-R0 16MHZ

Commit message: Started v2 update process.
Parts:
- removed U$9: MICRO-FIT_3.0_4POS_VERT_THRU, Schuyler:MICRO-FIT_3.0_4POS_VERT_THRU
- added U$15: MICRO-FIT_3.0_5POS_VERT_THRU, Schuyler:MICRO-FIT_3.0_5POS_VERT_THRU
- C13, C14, C15, C16, C17: value 0.1 uF -> 0.1uF
- JP2: value (none) -> M023.5MM
- U$2: value CC3-4805SF-ECC3-4805SF-E -> CC3-4805SF-E"; device Schuyler:CC3-4805SF-ECC3-4805SF-E -> Schuyler:CC3-4805SF-E"
- U$4: device Schuyler:MCP73831/2MCP73831/2 -> Schuyler:MCP73831/2'
- U3: device SparkFun:HEX_CONVERTER -> SparkFun-DigitalIC:HEX_CONVERTER
Connections:
- net 3.3V renamed 3V3
- new net SPEC_TRIGGER: U$15.P$5
- net +5V: now also U$15.P$1; no longer JP1.6, U$9.P$1
- net ARDUINO_V: now also JP1.6
- net GND: now also U$15.P$2; no longer U$9.P$2
- net RX_FROM_SPEC: now also U$15.P$4; no longer U$9.P$4
- net TX_TO_SPEC: now also U$15.P$3; no longer U$9.P$3
Other:
- note added: "NOTE: FIX SDO net"
- moved on the sheet: C10, C13, C14, C15, C16, C17, R8, TP4, U$1

Commit message: some continuing updates
Parts:
- removed JP1: (no value), pinhead:PINHD-1X7
- added C21: 0.1uF, resistor:C-USC0603
- added R22: 10k, SparkFun-Passives:RESISTOR0603-RES
- added U$20: BATTERY_12MM, Schuyler:BATTERY_12MM
- added U2: DS3234, Schuyler:DS3234
- C10, C12: value 4.7 uF -> 4.7uF
- C2, C8: SUPPLIER (none) -> DIGIKEY
- R3, R4, R5, R6: value (none) -> DNP
- R8: value (none) -> 20k
- U$1: value CC6-4812SF-ECC6-4812SF-E -> CC6-4812SF-E'; device Schuyler:CC6-4812SF-ECC6-4812SF-E -> Schuyler:CC6-4812SF-E'
Connections:
- removed net +5V: C12.1, C13.1, C16.1, C2.1, C8.1, IC1A.-TR, IC1A.RES, R10.2, R5.2, R9.2, TP6.TP, U$10.P$1, U$15.P$1, U$2.V_OUT+, U$4.VDD, U$6.A, U$7.IN, U$8.SHDN, U$8.VCC
- new net 5V0: C12.1, C13.1, C16.1, C2.1, C8.1, R5.2, R9.2, TP6.TP, U$10.P$1, U$15.P$1, U$2.V_OUT+, U$4.VDD, U$6.A, U$7.IN, U$8.SHDN, U$8.VCC
- new net N$20: R3.1, R4.2, U$1.TRM
- net 12V: now also R3.2; no longer R3.1
- net ARDUINO_V: now also C21.1, IC1A.-TR, IC1A.RES, R10.2, R22.2, U2.VCC; no longer JP1.6
- net GND: now also C21.2, U$20.V-, U2.GND, U2.NC@1, U2.NC@2, U2.NC@3, U2.NC@4, U2.NC@5, U2.NC@6, U2.NC@7, U2.NC@8, U2.NC@9; no longer JP1.7
- net IO3: now also R22.1, U2.!INT!/SQW; no longer JP1.5
- net IO9: now also U2.!CS; no longer JP1.1
- net MISO_IO12: now also U2.DOUT; no longer JP1.3
- net MOSI_IO11: now also U2.DIN; no longer JP1.2
- net N$6: now also U$20.V+, U2.VBAT; no longer R3.2, R4.2, U$1.TRM
- net SCK_IO13: now also U2.SCLK@1, U2.SCLK@2; no longer JP1.4
Other:
- note added: "Real Time Clock"
- note removed: "MISO"
- note removed: "MOSI"
- note removed: "RTC Connector"
- note removed: "SQW"
- note removed: "SS"
- note removed: "VCC"
- moved on the sheet: C1, C10, C12, C15, C16, C17, C19, C2, C20, C3, C6, C7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

Commit message: Version 2.0 Complete
Parts:
- removed IC1: 4098D, 40xx:4098D
- removed JP2: M023.5MM, SparkFun-Connectors:M023.5MM
- removed U$1: CC6-4812SF-E', Schuyler:CC6-4812SF-E'
- removed U$10: MICRO-FIT_3.0_7POS_VERT_THRU, Schuyler:MICRO-FIT_3.0_7POS_VERT_THRU
- removed U$11: GM1WA55321ACOMMON_CATHODE, Schuyler:GM1WA55321ACOMMON_CATHODE
- removed U$12, U$13: MICRO-FIT_3.0_2POS_VERT_THRU, Schuyler:MICRO-FIT_3.0_2POS_VERT_THRU
- removed U$14: MICRO-FIT_3.0_6POS_VERT_THRU, Schuyler:MICRO-FIT_3.0_6POS_VERT_THRU
- removed U$15: MICRO-FIT_3.0_5POS_VERT_THRU, Schuyler:MICRO-FIT_3.0_5POS_VERT_THRU
- removed U$2: CC3-4805SF-E", Schuyler:CC3-4805SF-E"
- removed U$20: BATTERY_12MM, Schuyler:BATTERY_12MM
- removed U$3: RF201L2S, Schuyler:RF201L2SRF201L2S
- removed U$4: MCP73831/2, Schuyler:MCP73831/2'
- removed U$5, U$6: LSM115J, Schuyler:LSM115JLSM115J
- removed U$7: LM3480IM4, SparkFun-PowerIC:LM3480IM4
- removed U$8: MAX3311, Schuyler:MAX3311MAX3311EEUB+
- removed Y2: CSTCE16M0V53-R0 16MHZ, SmartPrj:RESONATORMU
- removed ZU4: ATMEGA328P-PU, SmartPrj:ATMEGA328P-PU
- added B1: BATTERY_12MM, Schuyler:BATTERY_12MM
- added C23, C24: 0.1uF, resistor:C-USC0603
- added C25: 1uF, rcl:C-USC1206
- added D1: RF201L2S, Schuyler:RF201L2SRF201L2S
- added D3: LSM115J, Schuyler:LSM115JLSM115J
- added D4: RGB_LED_COMMON_ANODE_1, Schuyler:RGB_LED_COMMON_ANODE_1
- added J1: M023.5MM, SparkFun-Connectors:M023.5MM
- added J2, J3: MICRO-FIT_3.0_2POS_VERT_THRU, Schuyler:MICRO-FIT_3.0_2POS_VERT_THRU
- added J4: MICRO-FIT_3.0_7POS_VERT_THRU, Schuyler:MICRO-FIT_3.0_7POS_VERT_THRU
- added J5: MICRO-FIT_3.0_6POS_VERT_THRU, Schuyler:MICRO-FIT_3.0_6POS_VERT_THRU
- added J6: MICRO-FIT_3.0_5POS_VERT_THRU, Schuyler:MICRO-FIT_3.0_5POS_VERT_THRU
- added SD: MICRO_SD_DM3AT, Schuyler:MICRO_SD_DM3AT
- added U10: MULTIVIBRATOR_DUAL, Schuyler:MULTIVIBRATOR_DUAL
- added U4: CC6-4812SF-E', Schuyler:CC6-4812SF-E'
- added U5: CC3-4805SF-E", Schuyler:CC3-4805SF-E"
- added U6: HEX_CONVERTERS, Schuyler:HEX_CONVERTERS
- added U8: ST232, Schuyler:ST232
- added U9: ATMEGA328P-PU, SmartPrj:ATMEGA328P-PU
- added Y1: CSTCE16M0V53-R0 16MHZ, SmartPrj:RESONATORMU
- C1: value 1uF -> 4.7uF; device rcl:C-USC1206 -> resistor:C-USC0603; PARTNUMBER (none) -> 445-5178-1-ND; SUPPLIER (none) -> DIGIKEY
- C10: PARTNUMBER (none) -> 445-5178-1-ND; SUPPLIER (none) -> DIGIKEY
- C11: value 100n -> 0.1uF; device SmartPrj:C-EU0603-RND -> rcl:C-USC0603; PARTNUMBER (none) -> 311-1523-1-ND
- C12: value 4.7uF -> 1uF; device resistor:C-USC0603 -> rcl:C-USC1206; PARTNUMBER (none) -> 1276-2747-1-ND; SUPPLIER (none) -> DIGIKEY
- C13: value 0.1uF -> 1uF; device resistor:C-USC0603 -> rcl:C-USC1206; PARTNUMBER (none) -> 1276-2747-1-ND; SUPPLIER (none) -> DIGIKEY
- C14, C15: device resistor:C-USC0603 -> rcl:C-USC0603; PARTNUMBER (none) -> 311-1523-1-ND
- C16, C17, C5: PARTNUMBER (none) -> 311-1523-1-ND
- C18: value 1uF -> 0.1uF; PARTNUMBER (none) -> 311-1523-1-ND
- C19, C20: value 100nF -> 0.1uF; device rcl:C-USC0603 -> resistor:C-USC0603; PARTNUMBER (none) -> 311-1523-1-ND
- C2: value 1uF -> 0.1uF; device rcl:C-USC1206 -> resistor:C-USC0603; PARTNUMBER (none) -> 311-1523-1-ND; SUPPLIER DIGIKEY -> (none)
- C21: PARTNUMBER 399-1095-1-ND -> 311-1523-1-ND
- C3, C4: value 1uF -> 0.1uF; device rcl:C-USC1206 -> rcl:C-USC0603; PARTNUMBER (none) -> 311-1523-1-ND
- C6, C7: value 0.1uF -> 1uF; device rcl:C-USC0603 -> rcl:C-USC1206; PARTNUMBER (none) -> 1276-2747-1-ND; SUPPLIER (none) -> DIGIKEY
- C8: device rcl:C-USC0603 -> resistor:C-USC0603; PARTNUMBER (none) -> 311-1523-1-ND; SUPPLIER DIGIKEY -> (none)
- C9: value 100n -> 0.1uF; device SmartPrj:C-EU0603-RND -> resistor:C-USC0603; PARTNUMBER (none) -> 311-1523-1-ND
- D2: value CD1206-S01575 -> LSM115J; device diode:DIODE-MINIMELF -> Schuyler:LSM115JLSM115J
- R1: value (none) -> 4.99M
- R10: value 10k -> DNP
- R11: value 600 -> DNP
- R12: value 400 -> DNP
- R13: value 420 -> DNP
- R14: value 4.99M -> 33k
- R15: value 100k -> 33k
- R16: value 250k -> 33k
- R17: value 75k -> 10k
- R18: value (none) -> 1M; device SparkFun-Passives:RESISTOR0603-RES -> SmartPrj:R-EU_R0603; PARTNUMBER (none) -> P1.00MHCT-ND; SUPPLIER (none) -> DIGIKEY
- R19: value (none) -> 600
- R2: value (none) -> 100k
- R20: value (none) -> 360
- R21: value 10k -> 360
- R22: PARTNUMBER 311-10.0KHRCT-ND -> (none)
- R4: value DNP -> 10k; PARTNUMBER (none) -> 311-10.0KHRCT-ND
- R5, R6: value DNP -> 1k
- R7: value 1M -> 20k; device SmartPrj:R-EU_R0603 -> SparkFun-Passives:RESISTOR0603-RES
- R8: value 20k -> 250k
- R9: value 100k -> 75k
- S1: value (none) -> DIP03YL
- T1, T2: PARTNUMBER (none) -> MMBT2484LT1GOSCT-ND; SUPPLIER (none) -> DIGIKEY
- U1: value USD-SOCKETNEW -> DS3234; device SparkFun:USD-SOCKETNEW -> Schuyler:DS3234
- U2: value DS3234 -> LM3480IM4; device Schuyler:DS3234 -> SparkFun-PowerIC:LM3480IM4
- U3: value HEX_CONVERTER -> MCP73831/2; device SparkFun-DigitalIC:HEX_CONVERTER -> Schuyler:MCP73832
Connections:
- removed net N$11: C15.1, U$8.V-
- removed net N$12: C17.2, U$8.C1-
- removed net SPEC_TRIGGER: U$15.P$5
- new net N$19: C16.1, U8.C1+
- new net N$21: C16.2, U8.C1-
- new net N$22: C17.1, U8.C2+
- new net N$23: C17.2, U8.C2-
- new net N$24: C19.1, U8.V-
- new net N$26: C18.2, U8.V+
- net 12V: now also C12.1, C14.1, J5.P$1, R10.2, U4.V_OUT+; no longer C1.1, C7.1, R3.2, U$1.V_OUT+, U$14.P$1
- net 3.7BATT: now also D2.A, J3.P$1, R8.2, U3.V_BAT; no longer R16.2, U$13.P$1, U$4.V_BAT, U$5.A
- net 3V3: now also C8.1, SD.VDD, U2.OUT, U6.VCC; no longer C14.1, U$7.OUT, U1.VCC, U3.VCC
- net 48V: now also C7.1, D1.C, R1.2, U4.V_IN+, U5.V_IN+; no longer C3.1, R14.2, U$1.V_IN+, U$2.V_IN+, U$3.C
- net 48_V_BATTERY: now also D1.A, J1.1, J2.P$1; no longer JP2.1, U$12.P$1, U$3.A
- net 5V0: now also C1.1, C15.1, C18.1, C20.1, D3.A, J4.P$1, J6.P$1, R12.2, U2.IN, U3.VDD, U5.V_OUT+, U8.VCC; no longer C12.1, C16.1, C8.1, R5.2, R9.2, U$10.P$1, U$15.P$1, U$2.V_OUT+, U$4.VDD, U$6.A, U$7.IN, U$8.SHDN, U$8.VCC
- net AD0: now also U6.1A, U9.(ADC0)PC0); no longer R1.1, ZU4.(ADC0)PC0)
- net AD1: now also U1.!CS, U9.(ADC1)PC1; no longer R2.1, ZU4.(ADC1)PC1
- net AD2: now also R21.2, U9.(ADC2)PC2; no longer R12.2, ZU4.(ADC2)PC2
- net AD3: now also R20.2, U9.(ADC3)PC3; no longer R13.2, ZU4.(ADC3)PC3
- net AD4/SDA: now also C3.1, R1.1, R2.2, U9.(ADC4)PC4; no longer C19.1, R14.1, R15.2, ZU4.(ADC4)PC4
- net AD5/SCL: now also C11.1, R8.1, R9.2, U9.(ADC5)PC5; no longer C20.1, R16.1, R17.2, ZU4.(ADC5)PC5
- net ARDUINO_V: now also C24.1, C9.1, D3.C, D4.ANODE, R17.2, R4.2, U1.VCC, U10.!RES1, U10.-TR1, U10.VDD, U9.AVCC, U9.VCC; no longer C11.2, IC1A.-TR, IC1A.RES, R10.2, R21.2, U$5.C, U$6.C, U2.VCC, ZU4.AVCC, ZU4.VCC
- net AREF: now also C23.2, U9.AREF; no longer C9.2, ZU4.AREF
- net DEUTERIUM_ENABLE: now also J5.P$4, R14.2; no longer R18.2, U$14.P$4
- net GND: now also B1.V-, C11.2, C23.1, C24.2, C9.2, J1.2, J2.P$2, J3.P$2, J4.P$2, J5.P$2, J6.P$2, R11.1, R13.1, R14.1, R16.1, R2.1, R7.1, R9.1, SD.MOUNT, SD.VSS, U1.NC@1, U1.NC@2, U1.NC@3, U1.NC@4, U1.NC@5, U1.NC@6, U1.NC@7, U1.NC@8, U1.NC@9, U10.!RES2, U10.VSS, U3.VSS, U4.V_IN-, U4.V_OUT-, U5.V_IN-, U5.V_OUT-, U6.GND, U8.GND, U9.AGND, U9.GND, Y1.2; no longer C11.1, C16.2, C9.1, IC1B.RES, JP2.2, R17.1, R18.1, R19.1, R20.1, R4.1, R6.1, R8.1, U$1.V_IN-, U$1.V_OUT-, U$10.P$2, U$11.CATHODE, U$12.P$2, U$13.P$2, U$14.P$2, U$15.P$2, U$2.V_IN-, U$2.V_OUT-, U$20.V-, U$4.VSS, U$7.GND, U$8.GND, U1.SHIELD@1, U1.SHIELD@2, U1.SHIELD@3, U1.SHIELD@4, U2.NC@1, U2.NC@2, U2.NC@3, U2.NC@4, U2.NC@5, U2.NC@6, U2.NC@7, U2.NC@8, U2.NC@9, U3.GND, Y2.2, ZU4.AGND, ZU4.GND
- net IO2: now also J4.P$6, U9.(INT0)PD2; no longer R9.1, U$4.STAT, ZU4.(INT0)PD2
- net IO3: now also R3.2, R4.1, U1.!INT!/SQW, U9.(INT1)PD3; no longer R22.1, U2.!INT!/SQW, ZU4.(INT1)PD3
- net IO4: now also J6.P$5, U9.(T0)PD4; no longer U$10.P$5, ZU4.(T0)PD4
- net IO5: now also J4.P$5, U9.(T1)PD5; no longer U$10.P$6, ZU4.(T1)PD5
- net IO6: now also U10.+TR1, U9.(AIN0)PD6; no longer IC1A.+TR, ZU4.(AIN0)PD6
- net IO7: now also R19.2, U9.(AIN1)PD7; no longer R11.2, ZU4.(AIN1)PD7
- net IO8: now also R5.1, U9.(ICP)PB0; no longer U3.1A, ZU4.(ICP)PB0
- net IO9: now also R6.1, U9.(OC1)PB1; no longer U2.!CS, ZU4.(OC1)PB1
- net LAMP_5V: now also J5.P$3; no longer U$14.P$3
- net MISO_IO12: now also SD.DAT0, U1.DOUT, U9.(MISO)PB4; no longer U1.DO, U2.DOUT, ZU4.(MISO)PB4
- net MOSI_IO11: now also J4.P$3, U1.DIN, U6.2A, U9.(MOSI)PB3; no longer U$10.P$3, U2.DIN, U3.2A, ZU4.(MOSI)PB3
- net N$1: now also T2.C, U5.RC; no longer T1.C, U$2.RC
- net N$10: now also R3.1, U3.STAT; no longer C17.1, U$8.C1+
- net N$13: now also C25.2, U10.C1; no longer C18.2, IC1A.C
- net N$14: now also C25.1, R22.1, U10.R/C1; no longer C18.1, IC1A.R/C, R10.1
- net N$15: now also D4.RED, R19.1; no longer R11.1, U$11.RED
- net N$16: now also J4.P$7; no longer U$10.P$7
- net N$163: now also SD.DAT3, U6.1Y; no longer U1.CS, U3.1Y
- net N$17: now also D4.GREEN, R20.1; no longer R12.1, U$11.GREEN
- net N$18: now also D4.BLUE, R21.1; no longer R13.1, U$11.BLUE
- net N$2: now also T1.C, U4.RC; no longer T2.C, U$1.RC
- net N$20: now also R10.1, R11.2, U4.TRM; no longer R3.1, R4.2, U$1.TRM
- net N$3: now also R5.2, T1.B; no longer R2.2, T2.B
- net N$4: now also R6.2, T2.B; no longer R1.2, T1.B
- net N$5: now also R12.1, R13.2, U5.TRM; no longer R5.1, R6.2, U$2.TRM
- net N$6: now also B1.V+, U1.VBAT; no longer U$20.V+, U2.VBAT
- net N$7: now also R7.2, U3.PROG; no longer R8.2, U$4.PROG
- net N$8: now also SD.CMD, U6.2Y; no longer U1.DI, U3.2Y
- net N$9: now also SD.CLK, U6.3Y; no longer U1.SCK, U3.3Y
- net RESET: now also R17.1, U10.!Q1, U9.RESET; no longer D2.A, IC1A.!Q, R21.1, ZU4.RESET
- net RX_FROM_SPEC: now also J6.P$4, U8.R1IN; no longer U$15.P$4, U$8.RIN
- net RX_IO0: now also U8.R1OUT, U9.(RXD)PD0; no longer U$8.ROUT, ZU4.(RXD)PD0
- net SCK_IO13: now also J4.P$4, U1.SCLK@1, U1.SCLK@2, U6.3A, U9.(SCK)PB5; no longer U$10.P$4, U2.SCLK@1, U2.SCLK@2, U3.3A, ZU4.(SCK)PB5
- net SHUTTER_ENABLE: now also J5.P$6, R16.2; no longer R20.2, U$14.P$6
- net SS_IO10: now also U9.(SS)PB2; no longer ZU4.(SS)PB2
- net TUNGSTEN_ENABLE: now also J5.P$5, R15.2; no longer R19.2, U$14.P$5
- net TX_IO1: now also U8.T1IN, U9.(TXD)PD1; no longer U$8.TIN, ZU4.(TXD)PD1
- net TX_TO_SPEC: now also J6.P$3, U8.T1OUT; no longer U$15.P$3, U$8.TOUT
- net XTAL1: now also R18.1, U9.XTAL1, Y1.3; no longer R7.1, Y2.3, ZU4.XTAL1
- net XTAL2: now also R18.2, U9.XTAL2, Y1.1; no longer R7.2, Y2.1, ZU4.XTAL2
Other:
- moved on the sheet: C1, C10, C11, C12, C13, C14, C15, C16, C17, C18, C19, C2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

Commit message: Updated part attributes for ordering
Parts:
- J1: MANPARTNUMBER (none) -> 1984617; MANUFACTURER (none) -> Phoenix Contact; PARTNUMBER (none) -> 277-1721-ND; SUPPLIER (none) -> DIGIKEY
- R1: value 4.99M -> 5.1M; PARTNUMBER (none) -> 541-5.10MHCT-ND; SUPPLIER (none) -> DIGIKEY
- R14, R15, R16: PARTNUMBER (none) -> 311-33KGRCT-ND; SUPPLIER (none) -> DIGIKEY
- R17, R22: PARTNUMBER (none) -> 311-10.0KHRCT-ND; SUPPLIER (none) -> DIGIKEY
- R19: value 600 -> 604; PARTNUMBER (none) -> 1276-3506-1-ND; SUPPLIER (none) -> DIGIKEY
- R2: PARTNUMBER (none) -> 1276-3486-1-ND; SUPPLIER (none) -> DIGIKEY
- R20, R21: PARTNUMBER (none) -> 1276-5051-1-ND; SUPPLIER (none) -> DIGIKEY
- R4: SUPPLIER (none) -> DIGIKEY
- R5, R6: PARTNUMBER (none) -> 1276-5062-1-ND; SUPPLIER (none) -> DIGIKEY
- R7: PARTNUMBER (none) -> 1276-4768-1-ND; SUPPLIER (none) -> DIGIKEY
- R8: value 250k -> 249k; PARTNUMBER (none) -> 311-249KHRCT-ND; SUPPLIER (none) -> DIGIKEY
- R9: PARTNUMBER (none) -> 311-75.0KHRCT-ND; SUPPLIER (none) -> DIGIKEY
- RESET: PARTNUMBER (none) -> 450-1759-1-ND; SUPPLIER (none) -> DIGIKEY
- U9: PARTNUMBER (none) -> ATMEGA328P-PN-ND; SUPPLIER (none) -> DIGIKEY
